File: ZSWatch-kicad-v2/ZSWatch.kicad_pcb (KiCad board)
At the start: 4 copper layers, 41 x 38 mm, 73 parts, among them IC1 ESDALC6V1W5, IC2 XC9265C181MR-G, IC3 TPS61023DRLT, IC4 MAX30101EFD+T, IC5 FAN5622SX, IC6 BMI270, IC7 LIS2MDLTR, J2 Charger and programming heade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, M1 Vibrator DC Motor, U1 MAX1811ESA+, U10 0_NORA-B106, U11 TXB0104QRUTRQ1/NTS0104GU12, U13 GC9A01A_CST816S, U2 DMC2400UV-7, U3 NCV300LSN36T1G, U4 BMP581, U5 BME688, U6 DRV2603RUNT, U7 XC9265A331MR-G

Commit message: test differences
Parts:
- moved R5 1.92 mm to (103.2, 99.3)
Routing:
- net GND: track 107.9 -> 109.6 mm
